Commit message: new urdf

File: urdf/seven_dof_arm.urdf (robot description, URDF)
Before this commit: robot seven_dof_arm, 18 links, 17 joints
Links:
- removed link rgbd_camera_depth_frame
- removed link rgbd_camera_depth_optical_frame
- removed link rgbd_camera_link
- removed link rgbd_camera_optical_frame
- removed link rgbd_camera_rgb_frame
- removed link rgbd_camera_rgb_optical_frame
- link grasping_frame: geometry 
Joints:
- removed joint rgbd_camera_depth_joint
- removed joint rgbd_camera_depth_optical_joint
- removed joint rgbd_camera_joint
- removed joint rgbd_camera_optical_joint
- removed joint rgbd_camera_rgb_joint
- removed joint rgbd_camera_rgb_optical_joint
- joint gripper_roll_joint: limit lower=-2.61799387799 upper=2.6128806087 effort=300 velocity=1 -> lower=-3.14 upper=3.14 effort=300 velocity=1

File: urdf/seven_dof_arm.xacro (robot description, xacro)
@@ -365,5 +365,5 @@
       <origin xyz="0.04 0.03 0"/>
       <geometry>
-          <box size="${right_gripper_len} ${right_gripper_width} ${right_gripper_height}" />
+      	<box size="${right_gripper_len} ${right_gripper_width} ${right_gripper_height}" />
       </geometry>
       <material name="White" />
