Commit message: pan_tilt currently working for ROS2

File: urdf/pan_tilt.xacro (robot description, xacro)
@@ -43,5 +43,5 @@
     <axis xyz="0 0 1" />
     <limit effort="300" velocity="0.1" lower="-3.14" upper="3.14"/>
-    <dynamics damping="50" friction="1"/>
+    <dynamics damping="5" friction="1"/>
   </joint>
   <link name="pan_link">
@@ -69,5 +69,5 @@
     <axis xyz="0 1 0" />
     <limit effort="300" velocity="0.1" lower="-4.64" upper="-1.5"/>
-    <dynamics damping="50" friction="1"/>
+    <dynamics damping="5" friction="1"/>
   </joint>
   <link name="tilt_link">
@@ -89,3 +89,13 @@
 	<xacro:inertial_matrix mass="1"/>
   </link>
+	<gazebo>
+		<plugin name="joint_state_publisher" filename="libgazebo_ros_joint_state_publisher.so">
+      <ros>
+        <remapping>~/out:=joint_states</remapping>
+      </ros>
+      <update_rate>30</update_rate>
+      <joint_name>pan_joint</joint_name>
+      <joint_name>tilt_joint</joint_name>
+    </plugin>
+	</gazebo>
 </robot>
