Commit message: new functionality from ch11

File: urdf/sensors/xtion_pro_live.gazebo.xacro (robot description, xacro)
@@ -11,10 +11,10 @@
           <image>
             <format>R8G8B8</format>
-            <width>320</width>
-            <height>240</height>
+            <width>800</width>
+            <height>600</height>
           </image>
           <clip>
             <near>0.05</near>
-            <far>4.0</far>
+            <far>0.5</far>
           </clip>
         </camera>
@@ -31,5 +31,5 @@
           <pointCloudCutoff>0.05</pointCloudCutoff>
           <pointCloudCutoffMax>5</pointCloudCutoffMax>
-          <rangeMax>4.0</rangeMax>
+          <rangeMax>0.5</rangeMax>
           <!-- Distortion parameters not supported in gazebo 1.9.* plugins -->
           <!--distortionK1>0.00000001</distortionK1>
@@ -48,10 +48,10 @@
           <image>
             <format>R8G8B8</format>
-            <width>320</width>
-            <height>240</height>
+            <width>800</width>
+            <height>600</height>
           </image>
           <clip>
             <near>0.05</near>
-            <far>4.0</far>
+            <far>0.5</far>
           </clip>
         </camera>
@@ -68,5 +68,5 @@
           <pointCloudCutoff>0.05</pointCloudCutoff>
           <pointCloudCutoffMax>5</pointCloudCutoffMax>
-          <rangeMax>4.0</rangeMax>
+          <rangeMax>0.5</rangeMax>
         </plugin>
      </sensor>

File: urdf/seven_dof_arm.xacro (robot description, xacro)
@@ -295,5 +295,8 @@
     <origin xyz="0 0 0.080" rpy="${1.5*M_PI} -${.5*M_PI} 0" />
     <axis xyz="1 0 0" />
-    <limit effort="300" velocity="1" lower="-2.61799387799" upper="2.6128806087" />
+    <!--
+		<limit effort="300" velocity="1" lower="-2.61799387799" upper="2.6128806087" />
+		-->
+		<limit effort="300" velocity="1" lower="-3.14" upper="3.14" />
     <dynamics damping="50" friction="1"/>
   </joint>
@@ -382,5 +385,7 @@
       <origin xyz="0 0 0"/>
       <geometry>
+					<!--
           <box size="${grasp_frame_len} ${grasp_frame_width} ${grasp_frame_height}" />
+					-->
       </geometry>
       <material name="White" />

File: urdf/seven_dof_arm_with_rgbd.xacro (robot description, xacro)
@@ -371,5 +371,5 @@
     <material>Gazebo/White</material>
   </gazebo>
-    <!-- Grasping frame -->
+		<!--
     <link name="grasping_frame">
       <inertial>
@@ -392,4 +392,5 @@
       <origin xyz="0.08 0 0" rpy="0 0 0"/>
     </joint>
+		-->
   <xacro:include filename="$(find mastering_ros_robot_description_pkg)/urdf/sensors/xtion_pro_live.urdf.xacro"/>
 <!-- ///////////////////////////////////////////////////////////////////////////////////////////////////////////////////// -->
@@ -412,5 +413,5 @@
   <!-- Define RGB-D sensor -->
   <xacro:xtion_pro_live name="rgbd_camera" parent="base">
-    <origin xyz="0.1 0 1" rpy="0 ${75.0 * deg_to_rad} 0"/>
+    <origin xyz="0.15 0.0 0.8" rpy="0 ${75.0 * deg_to_rad} 0"/>
     <origin xyz="0 0 0" rpy="${-90.0 * deg_to_rad} 0 ${-90.0 * deg_to_rad}"/>
   </xacro:xtion_pro_live>
